File: Projeto_Placa_de_rele/Projeto_Placa_de_rele.kicad_sch (KiCad schematic)
At the start: 0 parts

Commit message: Atualização
Parts:
- added D1: 1N4007, Diode_THT:D_DO-41_SOD81_P10.16mm_Horizontal, symbol Device:D_Filled
- added D2: Red, LED_THT:LED_D5.0mm, symbol Device:LED_Filled
- added J1: Screw_Terminal_01x03, symbol Connector:Screw_Terminal_01x03
- added J2: Conn_01x03, Connector_PinHeader_2.54mm:PinHeader_1x03_P2.54mm_Vertical, symbol Connector_Generic:Conn_01x03
- added K1: SRD-05VDC-SL-C, Relay_THT:Relay_SPDT_Finder_36.11, symbol Relay:Relay_SPDT
- added Q1: BC547, Package_TO_SOT_THT:TO-92_Inline, symbol Transistor_BJT:Q_NPN_CBE
- added R1, R2: 470, Resistor_THT:R_Axial_DIN0207_L6.3mm_D2.5mm_P10.16mm_Horizontal, symbol Device:R
Connections:
- new net: D2.2 (A), R2.1
- new net +5V: D1.1 (K), J2.3 (Pin_3), K1.A1
- new net BASE: Q1.2 (B), R1.2
- new net COL: D1.2 (A), K1.A2, Q1.1 (C)
- new net GND: D2.1 (K), J2.1 (Pin_1), Q1.3 (E)
- new net RL_COM: J1.2 (Pin_2), K1.11
- new net RL_NC: J1.3 (Pin_3), K1.12
- new net RL_NO: J1.1 (Pin_1), K1.14
- new net SIG: J2.2 (Pin_2), R1.1, R2.2

Commit message: Atualização
Parts:
- J2: renamed from J1; footprint (none) -> TerminalBlock_Phoenix:TerminalBlock_Phoenix_MKDS-1,5-3-5.08_1x03_P5.08mm_Horizontal
- renumbered D2 to D1, D1 to D2, J2 to J1, R2 to R1, R1 to R2
Other:
- moved on the sheet: J2
Changed lines of the file:
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@@
 	(wire
 		(pts
-			(xy 190.5 67.31) (xy 203.2 67.31)
+			(xy 199.39 77.47) (xy 212.09 77.47)
 		)
 		(stroke
@@
 	(wire
 		(pts
-			(xy 190.5 62.23) (xy 203.2 62.23)
+			(xy 199.39 72.39) (xy 212.09 72.39)
 		)
 		(stroke
@@
 	(wire
 		(pts
-			(xy 190.5 64.77) (xy 203.2 64.77)
+			(xy 199.39 74.93) (xy 212.09 74.93)
 		)
 		(stroke
@@
 	)
 	(label "RL_NO"
-		(at 190.5 62.23 0)
+		(at 199.39 72.39 0)
 		(effects
 			(font
@@
 	)
 	(label "RL_COM"
-		(at 190.5 64.77 0)
+		(at 199.39 74.93 0)
 		(effects
 			(font
@@
 	)
 	(label "RL_NC"
-		(at 190.5 67.31 0)
+		(at 199.39 77.47 0)
 		(effects
 			(font
@@
 		(dnp no)
 		(fields_autoplaced yes)
-		(property "Reference" "R2"
+		(property "Reference" "R1"
 			(at 119.38 105.4099 0)
 			(effects
@@
 			(project "Projeto_Placa_de_rele"
 				(path "/3c7d3961-7c69-43c8-9b44-4ec8d2a3ba3a"
-					(reference "R2")
+					(reference "R1")
 					(unit 1)
 				)
@@
 		(dnp no)
 		(fields_autoplaced yes)
-		(property "Reference" "#PWR02"
+		(property "Reference" "#PWR04"
 			(at 139.7 67.31 0)
 			(effects
@@
 			(project "Projeto_Placa_de_rele"
 				(path "/3c7d3961-7c69-43c8-9b44-4ec8d2a3ba3a"
-					(reference "#PWR02")
+					(reference "#PWR04")
 					(unit 1)
 				)
@@
 		(dnp no)
 		(fields_autoplaced yes)
-		(property "Reference" "#PWR04"
+		(property "Reference" "#PWR03"
 			(at 116.84 132.08 0)
 			(effects
@@
 			(project ""
 				(path "/3c7d3961-7c69-43c8-9b44-4ec8d2a3ba3a"
-					(reference "#PWR04")
+					(reference "#PWR03")
 					(unit 1)
 				)
@@
 	(symbol
 		(lib_id "Connector:Screw_Terminal_01x03")
-		(at 208.28 64.77 0)
+		(at 217.17 74.93 0)
 		(unit 1)
 		(exclude_from_sim no)
@@
 		(dnp no)
 		(fields_autoplaced yes)
-		(property "Reference" "J1"
-			(at 210.82 63.4999 0)
+		(property "Reference" "J2"
+			(at 219.71 73.6599 0)
 			(effects
 				(font
@@
 		)
 		(property "Value" "Screw_Terminal_01x03"
-			(at 210.82 66.0399 0)
+			(at 219.71 76.1999 0)
 			(effects
 				(font
@@
 			)
 		)
-		(property "Footprint" ""
-			(at 208.28 64.77 0)
+		(property "Footprint" "TerminalBlock_Phoenix:TerminalBlock_Phoenix_MKDS-1,5-3-5.08_1x03_P5.08mm_Horizontal"
+			(at 217.17 74.93 0)
 			(effects
 				(font
@@
 		)
 		(property "Datasheet" "~"
-			(at 208.28 64.77 0)
+			(at 217.17 74.93 0)
 			(effects
 				(font
@@
 		)
 		(property "Description" "Generic screw terminal, single row, 01x03, script generated (kicad-library-utils/schlib/autogen/connector/)"
-			(at 208.28 64.77 0)
+			(at 217.17 74.93 0)
 			(effects
 				(font
@@
 			(project ""
 				(path "/3c7d3961-7c69-43c8-9b44-4ec8d2a3ba3a"
-					(reference "J1")
+					(reference "J2")
 					(unit 1)
 				)
@@
 		(dnp no)
 		(fields_autoplaced yes)
-		(property "Reference" "D2"
+		(property "Reference" "D1"
 			(at 120.65 118.4274 90)
 			(effects
@@
 			(project ""
 				(path "/3c7d3961-7c69-43c8-9b44-4ec8d2a3ba3a"
-					(reference "D2")
+					(reference "D1")
 					(unit 1)
 				)
@@
 		(dnp no)
 		(fields_autoplaced yes)
-		(property "Reference" "#PWR03"
+		(property "Reference" "#PWR02"
 			(at 104.14 132.08 0)
 			(effects
@@
 			(project ""
 				(path "/3c7d3961-7c69-43c8-9b44-4ec8d2a3ba3a"
-					(reference "#PWR03")
+					(reference "#PWR02")
 					(unit 1)
 				)
@@
 		(dnp no)
 		(fields_autoplaced yes)
-		(property "Reference" "J2"
+		(property "Reference" "J1"
 			(at 96.52 91.44 0)
 			(effects
@@
 			(project ""
 				(path "/3c7d3961-7c69-43c8-9b44-4ec8d2a3ba3a"
-					(reference "J2")
+					(reference "J1")
 					(unit 1)
 				)
@@
 		(dnp no)
 		(fields_autoplaced yes)
-		(property "Reference" "D1"
+		(property "Reference" "D2"
 			(at 142.24 76.1999 90)
 			(effects
@@
 			(project ""
 				(path "/3c7d3961-7c69-43c8-9b44-4ec8d2a3ba3a"
-					(reference "D1")
+					(reference "D2")
 					(unit 1)
 				)
@@
 		(dnp no)
 		(fields_autoplaced yes)
-		(property "Reference" "R1"
+		(property "Reference" "R2"
 			(at 123.19 93.98 90)
 			(effects
@@
 			(project ""
 				(path "/3c7d3961-7c69-43c8-9b44-4ec8d2a3ba3a"
-					(reference "R1")
+					(reference "R2")
 					(unit 1)
 				)

Commit message: Atualização kicad10
Parts:
- Q1: footprint Package_TO_SOT_THT:TO-92_Inline -> Package_TO_SOT_THT:TO-92L_Inline_Wide
