File: Projeto_Placa_de_rele/Projeto_Placa_de_rele.kicad_pcb (KiCad board)
At the start: 2 copper layers, 8 parts, among them J1 Conn_01x03, J2 Screw_Terminal_01x03, K1 SRD-05VDC-SL-C, Q1 BC547

Commit message: Atualização
Parts:
- moved Q1 20.8 mm to (133.9, 93.3), turned to 90 degrees
- moved K1 15.5 mm to (138.9, 101.3)
- moved J1 11.8 mm to (142.0, 84.0), turned to 90 degrees
- moved R1 8.89 mm to (139.4, 89.5)
- moved R2 8.87 mm to (139.4, 93.5)
- moved D1 7.66 mm to (156.5, 88.7), turned to -90 degrees
- moved J2 4.99 mm to (140.0, 124.4)
- moved D2 4.64 mm to (134.0, 109.6), turned to 90 degrees
Other:
- board outline added: 35 x 50 mm

Commit message: Atualização kicad10
Parts:
- Q1: footprint Package_TO_SOT_THT:TO-92_Inline -> Package_TO_SOT_THT:TO-92L_Inline_Wide
- moved R2 10.3 mm to (149.7, 92.4), turned to 180 degrees
- moved R1 10.2 mm to (149.6, 88.4), turned to 180 degrees
- moved J1 5.02 mm to (147.0, 83.6), turned to -90 degrees
- moved Q1 1.28 mm to (133.8, 94.5)
- moved J2 0.18 mm to (139.8, 124.4)
Routing:
- net +5V: track 0.00 -> 51.6 mm
- net GND: track 0.00 -> 48.2 mm
- net /COL: track 0.00 -> 28.5 mm
- net /RL_COM: track 0.00 -> 25.4 mm
- net /SIG: track 0.00 -> 16.9 mm
- net /RL_NO: track 0.00 -> 11.4 mm
- net /RL_NC: track 0.00 -> 11.3 mm
- net Net-(D1-A): track 0.00 -> 7.92 mm
- net /BASE: track 0.00 -> 5.83 mm

Commit message: Atualização Placa Relé.
Routing:
- net /SIG: track 16.9 -> 20.4 mm
Other:
- board text added: "Project #1: Relay Board Version: v1.0.0 Data: 28/04/26"
