File: Projeto_2_Microcontrolador_ponteH/input12V.kicad_sch (KiCad schematic)
At the start: 6 parts, among them J1 Barrel_Jack_Switch

Commit message: Atualização
Parts:
- renumbered D1 to D?, D2 to D?, F1 to F?, J1 to J?, R1 to R?, RV1 to RV?
Changed lines of the file:
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@@
 		(dnp no)
 		(fields_autoplaced yes)
-		(property "Reference" "#PWR01"
+		(property "Reference" "#PWR?"
 			(at 135.89 111.76 0)
 			(hide yes)
@@
 			(project "Projeto_2_Microcontrolador_ponteH"
 				(path "/93a75674-771f-42db-996f-b6f244100914/fb7b8ca1-1fb8-418d-aabd-461e5afed239"
-					(reference "#PWR01")
+					(reference "#PWR?")
 					(unit 1)
 				)
@@
 		(dnp no)
 		(fields_autoplaced yes)
-		(property "Reference" "RV1"
+		(property "Reference" "RV?"
 			(at 139.7 86.1665 0)
 			(show_name no)
@@
 			(project "Projeto_2_Microcontrolador_ponteH"
 				(path "/93a75674-771f-42db-996f-b6f244100914/fb7b8ca1-1fb8-418d-aabd-461e5afed239"
-					(reference "RV1")
+					(reference "RV?")
 					(unit 1)
 				)
@@
 		(dnp no)
 		(fields_autoplaced yes)
-		(property "Reference" "F1"
+		(property "Reference" "F?"
 			(at 128.27 73.66 90)
 			(show_name no)
@@
 			(project "Projeto_2_Microcontrolador_ponteH"
 				(path "/93a75674-771f-42db-996f-b6f244100914/fb7b8ca1-1fb8-418d-aabd-461e5afed239"
-					(reference "F1")
+					(reference "F?")
 					(unit 1)
 				)
@@
 		(dnp no)
 		(fields_autoplaced yes)
-		(property "Reference" "#PWR02"
+		(property "Reference" "#PWR?"
 			(at 121.92 111.76 0)
 			(hide yes)
@@
 			(project "Projeto_2_Microcontrolador_ponteH"
 				(path "/93a75674-771f-42db-996f-b6f244100914/fb7b8ca1-1fb8-418d-aabd-461e5afed239"
-					(reference "#PWR02")
+					(reference "#PWR?")
 					(unit 1)
 				)
@@
 		(dnp no)
 		(fields_autoplaced yes)
-		(property "Reference" "J1"
+		(property "Reference" "J?"
 			(at 110.49 73.66 0)
 			(show_name no)
@@
 			(project "Projeto_2_Microcontrolador_ponteH"
 				(path "/93a75674-771f-42db-996f-b6f244100914/fb7b8ca1-1fb8-418d-aabd-461e5afed239"
-					(reference "J1")
+					(reference "J?")
 					(unit 1)
 				)
@@
 		(dnp no)
 		(fields_autoplaced yes)
-		(property "Reference" "D1"
+		(property "Reference" "D?"
 			(at 149.86 73.66 0)
 			(show_name no)
@@
 			(project "Projeto_2_Microcontrolador_ponteH"
 				(path "/93a75674-771f-42db-996f-b6f244100914/fb7b8ca1-1fb8-418d-aabd-461e5afed239"
-					(reference "D1")
+					(reference "D?")
 					(unit 1)
 				)
@@
 		(dnp no)
 		(fields_autoplaced yes)
-		(property "Reference" "R1"
+		(property "Reference" "R?"
 			(at 163.83 86.3599 0)
 			(show_name no)
@@
 			(project "Projeto_2_Microcontrolador_ponteH"
 				(path "/93a75674-771f-42db-996f-b6f244100914/fb7b8ca1-1fb8-418d-aabd-461e5afed239"
-					(reference "R1")
+					(reference "R?")
 					(unit 1)
 				)
@@
 		(in_pos_files yes)
 		(dnp no)
-		(property "Reference" "D2"
+		(property "Reference" "D?"
 			(at 155.194 98.298 0)
 			(show_name no)
@@
 			(project "Projeto_2_Microcontrolador_ponteH"
 				(path "/93a75674-771f-42db-996f-b6f244100914/fb7b8ca1-1fb8-418d-aabd-461e5afed239"
-					(reference "D2")
+					(reference "D?")
 					(unit 1)
 				)
@@
 		(dnp no)
 		(fields_autoplaced yes)
-		(property "Reference" "#PWR03"
+		(property "Reference" "#PWR?"
 			(at 161.29 111.76 0)
 			(hide yes)
@@
 			(project "Projeto_2_Microcontrolador_ponteH"
 				(path "/93a75674-771f-42db-996f-b6f244100914/fb7b8ca1-1fb8-418d-aabd-461e5afed239"
-					(reference "#PWR03")
-					(unit 1)
-				)
+					(reference "#PWR?")
+					(unit 1)
+				)
