File: Projeto_2_Microcontrolador_ponteH/interface.kicad_sch (KiCad schematic)
At the start: 0 parts

Commit message: Atualização
Parts:
- added C? (x4): C, symbol Device:C
- added D?: Green, symbol Device:LED_Filled
- added D?: Red, symbol Device:LED_Filled
- added R? (x10): R, symbol Device:R
- added SW? (x4): SW_Push, symbol Switch:SW_Push
Connections:
- new net: R?.1, R?.1, SW?.2 (x4)
- new net: D?.2 (A), R?.2 (x2)
- new net +3V3: R?.2, R?.2, R?.2, R?.2
- new net GND: C?.2, C?.2, C?.2, C?.2, D?.1 (K), D?.1 (K), SW?.1, SW?.1, SW?.1, SW?.1
- new net LED_ERROR: R?.1
- new net LED_STATE: R?.1
- new net sw_1: C?.1, R?.2
- new net sw_2: C?.1, R?.2
- new net sw_3: C?.1, R?.2
- new net sw_4: C?.1, R?.2
