File: Projeto_2_Microcontrolador_ponteH/mcu.kicad_sch (KiCad schematic)
At the start: 13 parts, among them J2 Conn_01x05, U1 STM32G031F6Px

Commit message: Atualização
Parts:
- renumbered C4 to C?, C3 to C?, J2 to J?, R2 to R?, R5 to R?, R4 to R?, R3 to R?, TP2 to TP?, TP1 to TP?, TP3 to TP?, TP5 to TP?, TP4 to TP?, U1 to U?
Changed lines of the file:
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@@
 		(dnp no)
 		(fields_autoplaced yes)
-		(property "Reference" "#PWR06"
+		(property "Reference" "#PWR?"
 			(at 140.97 135.89 0)
 			(hide yes)
@@
 			(project "Projeto_2_Microcontrolador_ponteH"
 				(path "/93a75674-771f-42db-996f-b6f244100914/4de3da96-660b-413c-99c9-762894d4c1b3"
-					(reference "#PWR06")
+					(reference "#PWR?")
 					(unit 1)
 				)
@@
 		(dnp no)
 		(fields_autoplaced yes)
-		(property "Reference" "TP2"
+		(property "Reference" "TP?"
 			(at 254 126.9999 90)
 			(show_name no)
@@
 			(project "Projeto_2_Microcontrolador_ponteH"
 				(path "/93a75674-771f-42db-996f-b6f244100914/4de3da96-660b-413c-99c9-762894d4c1b3"
-					(reference "TP2")
+					(reference "TP?")
 					(unit 1)
 				)
@@
 		(dnp no)
 		(fields_autoplaced yes)
-		(property "Reference" "#PWR08"
+		(property "Reference" "#PWR?"
 			(at 120.65 57.15 0)
 			(hide yes)
@@
 			(project "Projeto_2_Microcontrolador_ponteH"
 				(path "/93a75674-771f-42db-996f-b6f244100914/4de3da96-660b-413c-99c9-762894d4c1b3"
-					(reference "#PWR08")
+					(reference "#PWR?")
 					(unit 1)
 				)
@@
 		(dnp no)
 		(fields_autoplaced yes)
-		(property "Reference" "U1"
+		(property "Reference" "U?"
 			(at 143.1133 76.2 0)
 			(show_name no)
@@
 			(project "Projeto_2_Microcontrolador_ponteH"
 				(path "/93a75674-771f-42db-996f-b6f244100914/4de3da96-660b-413c-99c9-762894d4c1b3"
-					(reference "U1")
+					(reference "U?")
 					(unit 1)
 				)
@@
 		(dnp no)
 		(fields_autoplaced yes)
-		(property "Reference" "#PWR014"
+		(property "Reference" "#PWR?"
 			(at 234.95 154.94 0)
 			(hide yes)
@@
 			(project "Projeto_2_Microcontrolador_ponteH"
 				(path "/93a75674-771f-42db-996f-b6f244100914/4de3da96-660b-413c-99c9-762894d4c1b3"
-					(reference "#PWR014")
+					(reference "#PWR?")
 					(unit 1)
 				)
@@
 		(dnp no)
 		(fields_autoplaced yes)
-		(property "Reference" "J2"
+		(property "Reference" "J?"
 			(at 260.35 88.8999 0)
 			(show_name no)
@@
 			(project "Projeto_2_Microcontrolador_ponteH"
 				(path "/93a75674-771f-42db-996f-b6f244100914/4de3da96-660b-413c-99c9-762894d4c1b3"
-					(reference "J2")
+					(reference "J?")
 					(unit 1)
 				)
@@
 		(in_pos_files yes)
 		(dnp no)
-		(property "Reference" "R2"
+		(property "Reference" "R?"
 			(at 232.41 84.328 90)
 			(show_name no)
@@
 			(project "Projeto_2_Microcontrolador_ponteH"
 				(path "/93a75674-771f-42db-996f-b6f244100914/4de3da96-660b-413c-99c9-762894d4c1b3"
-					(reference "R2")
+					(reference "R?")
 					(unit 1)
 				)
@@
 		(dnp no)
 		(fields_autoplaced yes)
-		(property "Reference" "C4"
+		(property "Reference" "C?"
 			(at 124.46 39.3699 0)
 			(show_name no)
@@
 			(project "Projeto_2_Microcontrolador_ponteH"
 				(path "/93a75674-771f-42db-996f-b6f244100914/4de3da96-660b-413c-99c9-762894d4c1b3"
-					(reference "C4")
+					(reference "C?")
 					(unit 1)
 				)
@@
 		(dnp no)
 		(fields_autoplaced yes)
-		(property "Reference" "C3"
+		(property "Reference" "C?"
 			(at 110.49 39.3699 0)
 			(show_name no)
@@
 			(project "Projeto_2_Microcontrolador_ponteH"
 				(path "/93a75674-771f-42db-996f-b6f244100914/4de3da96-660b-413c-99c9-762894d4c1b3"
-					(reference "C3")
+					(reference "C?")
 					(unit 1)
 				)
@@
 		(in_pos_files yes)
 		(dnp no)
-		(property "Reference" "R5"
+		(property "Reference" "R?"
 			(at 222.758 80.01 90)
 			(show_name no)
@@
 			(project "Projeto_2_Microcontrolador_ponteH"
 				(path "/93a75674-771f-42db-996f-b6f244100914/4de3da96-660b-413c-99c9-762894d4c1b3"
-					(reference "R5")
+					(reference "R?")
 					(unit 1)
 				)
@@
 		(dnp no)
 		(fields_autoplaced yes)
-		(property "Reference" "TP1"
+		(property "Reference" "TP?"
 			(at 254 121.9199 90)
 			(show_name no)
@@
 			(project "Projeto_2_Microcontrolador_ponteH"
 				(path "/93a75674-771f-42db-996f-b6f244100914/4de3da96-660b-413c-99c9-762894d4c1b3"
-					(reference "TP1")
+					(reference "TP?")
 					(unit 1)
 				)
@@
 		(dnp no)
 		(fields_autoplaced yes)
-		(property "Reference" "#PWR013"
+		(property "Reference" "#PWR?"
 			(at 234.95 123.19 0)
 			(hide yes)
@@
 			(project "Projeto_2_Microcontrolador_ponteH"
 				(path "/93a75674-771f-42db-996f-b6f244100914/4de3da96-660b-413c-99c9-762894d4c1b3"
-					(reference "#PWR013")
+					(reference "#PWR?")
 					(unit 1)
 				)
@@
 		(dnp no)
 		(fields_autoplaced yes)
-		(property "Reference" "#PWR07"
+		(property "Reference" "#PWR?"
 			(at 140.97 74.93 0)
 			(hide yes)
@@
 			(project "Projeto_2_Microcontrolador_ponteH"
 				(path "/93a75674-771f-42db-996f-b6f244100914/4de3da96-660b-413c-99c9-762894d4c1b3"
-					(reference "#PWR07")
+					(reference "#PWR?")
 					(unit 1)
 				)
@@
 		(dnp no)
 		(fields_autoplaced yes)
-		(property "Reference" "#PWR09"
+		(property "Reference" "#PWR?"
 			(at 106.68 36.83 0)
 			(hide yes)
@@
 			(project "Projeto_2_Microcontrolador_ponteH"
 				(path "/93a75674-771f-42db-996f-b6f244100914/4de3da96-660b-413c-99c9-762894d4c1b3"
-					(reference "#PWR09")
+					(reference "#PWR?")
 					(unit 1)
 				)
@@
 		(dnp no)
 		(fields_autoplaced yes)
-		(property "Reference" "TP3"
+		(property "Reference" "TP?"
 			(at 254 132.0799 90)
 			(show_name no)
@@
 			(project "Projeto_2_Microcontrolador_ponteH"
 				(path "/93a75674-771f-42db-996f-b6f244100914/4de3da96-660b-413c-99c9-762894d4c1b3"
-					(reference "TP3")
+					(reference "TP?")
 					(unit 1)
 				)
@@
 		(in_pos_files yes)
 		(dnp no)
-		(property "Reference" "R4"
+		(property "Reference" "R?"
 			(at 232.41 97.028 90)
 			(show_name no)
@@
 			(project "Projeto_2_Microcontrolador_ponteH"
 				(path "/93a75674-771f-42db-996f-b6f244100914/4de3da96-660b-413c-99c9-762894d4c1b3"
-					(reference "R4")
+					(reference "R?")
 					(unit 1)
 				)
@@
 		(dnp no)
 		(fields_autoplaced yes)
-		(property "Reference" "TP5"
+		(property "Reference" "TP?"
 			(at 254 142.2399 90)
 			(show_name no)
@@
 			(project "Projeto_2_Microcontrolador_ponteH"
 				(path "/93a75674-771f-42db-996f-b6f244100914/4de3da96-660b-413c-99c9-762894d4c1b3"
-					(reference "TP5")
+					(reference "TP?")
 					(unit 1)
 				)
@@
 		(dnp no)
 		(fields_autoplaced yes)
-		(property "Reference" "#PWR010"
+		(property "Reference" "#PWR?"
 			(at 247.65 76.2 0)
 			(hide yes)
@@
 			(project "Projeto_2_Microcontrolador_ponteH"
 				(path "/93a75674-771f-42db-996f-b6f244100914/4de3da96-660b-413c-99c9-762894d4c1b3"
-					(reference "#PWR010")
+					(reference "#PWR?")
 					(unit 1)
 				)
@@
 		(dnp no)
 		(fields_autoplaced yes)
-		(property "Reference" "#PWR011"
+		(property "Reference" "#PWR?"
 			(at 247.65 107.95 0)
 			(hide yes)
@@
 			(project "Projeto_2_Microcontrolador_ponteH"
 				(path "/93a75674-771f-42db-996f-b6f244100914/4de3da96-660b-413c-99c9-762894d4c1b3"
-					(reference "#PWR011")
+					(reference "#PWR?")
 					(unit 1)
 				)
@@
 		(dnp no)
 		(fields_autoplaced yes)
-		(property "Reference" "#PWR012"
+		(property "Reference" "#PWR?"
 			(at 224.79 76.2 0)
 			(hide yes)
@@
 			(project "Projeto_2_Microcontrolador_ponteH"
 				(path "/93a75674-771f-42db-996f-b6f244100914/4de3da96-660b-413c-99c9-762894d4c1b3"
-					(reference "#PWR012")
+					(reference "#PWR?")
 					(unit 1)
 				)
@@
 		(dnp no)
 		(fields_autoplaced yes)
-		(property "Reference" "TP4"
+		(property "Reference" "TP?"
 			(at 254 137.1599 90)
 			(show_name no)
@@
 			(project "Projeto_2_Microcontrolador_ponteH"
 				(path "/93a75674-771f-42db-996f-b6f244100914/4de3da96-660b-413c-99c9-762894d4c1b3"
-					(reference "TP4")
+					(reference "TP?")
 					(unit 1)
 				)
@@
 		(in_pos_files yes)
 		(dnp no)
-		(property "Reference" "R3"
+		(property "Reference" "R?"
 			(at 232.41 90.678 90)
 			(show_name no)
@@
 			(project "Projeto_2_Microcontrolador_ponteH"
 				(path "/93a75674-771f-42db-996f-b6f244100914/4de3da96-660b-413c-99c9-762894d4c1b3"
-					(reference "R3")
-					(unit 1)
-				)
+					(reference "R?")
+					(unit 1)
+				)

Commit message: Atualização
Other:
- moved on the sheet: C?
Changed lines of the file:
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@@
 	(paper "A4")
 	(junction
-		(at 120.65 46.99)
-		(diameter 0)
-		(color 0 0 0 0)
-	)
-	(junction
-		(at 106.68 34.29)
+		(at 76.2 36.83)
 		(diameter 0)
 		(color 0 0 0 0)
@@
 		(color 0 0 0 0)
 	)
-	(wire
-		(pts
-			(xy 106.68 34.29) (xy 120.65 34.29)
-		)
-		(stroke
-			(width 0)
-			(type default)
-		)
-	)
-	(wire
-		(pts
-			(xy 120.65 44.45) (xy 120.65 46.99)
+	(junction
+		(at 76.2 46.99)
+		(diameter 0)
+		(color 0 0 0 0)
+	)
+	(wire
+		(pts
+			(xy 76.2 34.29) (xy 76.2 36.83)
 		)
 		(stroke
@@
 	(wire
 		(pts
-			(xy 120.65 34.29) (xy 120.65 36.83)
+			(xy 69.85 46.99) (xy 76.2 46.99)
 		)
 		(stroke
@@
 	(wire
 		(pts
+			(xy 76.2 36.83) (xy 82.55 36.83)
+		)
+		(stroke
+			(width 0)
+			(type default)
+		)
+	)
+	(wire
+		(pts
 			(xy 237.49 86.36) (xy 237.49 90.17)
 		)
@@
 	(wire
 		(pts
+			(xy 82.55 45.72) (xy 82.55 46.99)
+		)
+		(stroke
+			(width 0)
+			(type default)
+		)
+	)
+	(wire
+		(pts
 			(xy 237.49 99.06) (xy 237.49 95.25)
 		)
@@
 	(wire
 		(pts
-			(xy 106.68 33.02) (xy 106.68 34.29)
+			(xy 69.85 45.72) (xy 69.85 46.99)
 		)
 		(stroke
@@
 	(wire
 		(pts
-			(xy 106.68 46.99) (xy 120.65 46.99)
-		)
-		(stroke
-			(width 0)
-			(type default)
-		)
-	)
-	(wire
-		(pts
 			(xy 224.79 82.55) (xy 224.79 86.36)
 		)
@@
 	(wire
 		(pts
+			(xy 76.2 46.99) (xy 82.55 46.99)
+		)
+		(stroke
+			(width 0)
+			(type default)
+		)
+	)
+	(wire
+		(pts
 			(xy 212.09 99.06) (xy 229.87 99.06)
 		)
@@
 	(wire
 		(pts
+			(xy 69.85 38.1) (xy 69.85 36.83)
+		)
+		(stroke
+			(width 0)
+			(type default)
+		)
+	)
+	(wire
+		(pts
 			(xy 237.49 90.17) (xy 252.73 90.17)
 		)
@@
 	(wire
 		(pts
+			(xy 82.55 36.83) (xy 82.55 38.1)
+		)
+		(stroke
+			(width 0)
+			(type default)
+		)
+	)
+	(wire
+		(pts
 			(xy 234.95 128.27) (xy 248.92 128.27)
 		)
@@
 	(wire
 		(pts
-			(xy 120.65 46.99) (xy 120.65 50.8)
-		)
-		(stroke
-			(width 0)
-			(type default)
-		)
-	)
-	(wire
-		(pts
 			(xy 234.95 86.36) (xy 237.49 86.36)
 		)
@@
 	(wire
 		(pts
-			(xy 106.68 34.29) (xy 106.68 36.83)
-		)
-		(stroke
-			(width 0)
-			(type default)
-		)
-	)
-	(wire
-		(pts
 			(xy 234.95 123.19) (xy 248.92 123.19)
 		)
@@
 	(wire
 		(pts
-			(xy 106.68 44.45) (xy 106.68 46.99)
-		)
-		(stroke
-			(width 0)
-			(type default)
-		)
-	)
-	(wire
-		(pts
 			(xy 247.65 85.09) (xy 247.65 72.39)
 		)
@@
 	(wire
 		(pts
+			(xy 69.85 36.83) (xy 76.2 36.83)
+		)
+		(stroke
+			(width 0)
+			(type default)
+		)
+	)
+	(wire
+		(pts
 			(xy 212.09 86.36) (xy 224.79 86.36)
+		)
+		(stroke
+			(width 0)
+			(type default)
+		)
+	)
+	(wire
+		(pts
+			(xy 76.2 46.99) (xy 76.2 49.53)
 		)
 		(stroke
@@
 	(symbol
 		(lib_id "power:GND")
-		(at 120.65 50.8 0)
+		(at 76.2 49.53 0)
 		(unit 1)
 		(body_style 1)
@@
 		(fields_autoplaced yes)
 		(property "Reference" "#PWR?"
-			(at 120.65 57.15 0)
+			(at 76.2 55.88 0)
 			(hide yes)
 			(show_name no)
@@
 		)
 		(property "Value" "GND"
-			(at 120.65 55.88 0)
+			(at 76.2 54.61 0)
 			(show_name no)
 			(do_not_autoplace no)
@@
 		)
 		(property "Footprint" ""
-			(at 120.65 50.8 0)
+			(at 76.2 49.53 0)
 			(hide yes)
 			(show_name no)
@@
 		)
 		(property "Datasheet" ""
-			(at 120.65 50.8 0)
+			(at 76.2 49.53 0)
 			(hide yes)
 			(show_name no)
@@
 		)
 		(property "Description" "Power symbol creates a global label with name \"GND\" , ground"
-			(at 120.65 50.8 0)
+			(at 76.2 49.53 0)
 			(hide yes)
 			(show_name no)
@@
 	(symbol
 		(lib_id "Device:C")
-		(at 120.65 40.64 0)
+		(at 82.55 41.91 0)
 		(unit 1)
 		(body_style 1)
@@
 		(fields_autoplaced yes)
 		(property "Reference" "C?"
-			(at 124.46 39.3699 0)
+			(at 86.36 40.6399 0)
 			(show_name no)
 			(do_not_autoplace no)
@@
 		)
 		(property "Value" "C"
-			(at 124.46 41.9099 0)
+			(at 86.36 43.1799 0)
 			(show_name no)
 			(do_not_autoplace no)
@@
 		)
 		(property "Footprint" ""
-			(at 121.6152 44.45 0)
+			(at 83.5152 45.72 0)
 			(hide yes)
 			(show_name no)
@@
 		)
 		(property "Datasheet" ""
-			(at 120.65 40.64 0)
+			(at 82.55 41.91 0)
 			(hide yes)
 			(show_name no)
@@
 		)
 		(property "Description" "Unpolarized capacitor"
-			(at 120.65 40.64 0)
+			(at 82.55 41.91 0)
 			(hide yes)
 			(show_name no)
@@
 	(symbol
 		(lib_id "Device:C")
-		(at 106.68 40.64 0)
+		(at 69.85 41.91 0)
 		(unit 1)
 		(body_style 1)
@@
 		(fields_autoplaced yes)
 		(property "Reference" "C?"
-			(at 110.49 39.3699 0)
+			(at 73.66 40.6399 0)
 			(show_name no)
 			(do_not_autoplace no)
@@
 		)
 		(property "Value" "C"
-			(at 110.49 41.9099 0)
+			(at 73.66 43.1799 0)
 			(show_name no)
 			(do_not_autoplace no)
@@
 		)
 		(property "Footprint" ""
-			(at 107.6452 44.45 0)
+			(at 70.8152 45.72 0)
 			(hide yes)
 			(show_name no)
@@
 		)
 		(property "Datasheet" ""
-			(at 106.68 40.64 0)
+			(at 69.85 41.91 0)
 			(hide yes)
 			(show_name no)
@@
 		)
 		(property "Description" "Unpolarized capacitor"
-			(at 106.68 40.64 0)
+			(at 69.85 41.91 0)
 			(hide yes)
 			(show_name no)
@@
 	(symbol
 		(lib_id "power:+3V3")
-		(at 106.68 33.02 0)
+		(at 76.2 34.29 0)
 		(unit 1)
 		(body_style 1)
@@
 		(fields_autoplaced yes)
 		(property "Reference" "#PWR?"
-			(at 106.68 36.83 0)
+			(at 76.2 38.1 0)
 			(hide yes)
 			(show_name no)
@@
 		)
 		(property "Value" "+3V3"
-			(at 106.68 27.94 0)
+			(at 76.2 29.21 0)
 			(show_name no)
 			(do_not_autoplace no)
@@
 		)
 		(property "Footprint" ""
-			(at 106.68 33.02 0)
+			(at 76.2 34.29 0)
 			(hide yes)
 			(show_name no)
@@
 		)
 		(property "Datasheet" ""
-			(at 106.68 33.02 0)
+			(at 76.2 34.29 0)
 			(hide yes)
 			(show_name no)
@@
 		)
 		(property "Description" "Power symbol creates a global label with name \"+3V3\""
-			(at 106.68 33.02 0)
-			(hide yes)
-			(show_name no)
+			(at 76.2 34.29 0)
+			(hide yes)
+			(show_name no)
