File: Projeto_2_Microcontrolador_ponteH/Regulator_3_3V.kicad_sch (KiCad schematic)
At the start: 2 parts

Commit message: Atualização
Parts:
- renumbered C1 to C?, C2 to C?
Changed lines of the file:
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@@
 		(dnp no)
 		(fields_autoplaced yes)
-		(property "Reference" "#PWR05"
+		(property "Reference" "#PWR?"
 			(at 154.94 101.6 0)
 			(hide yes)
@@
 			(project "Projeto_2_Microcontrolador_ponteH"
 				(path "/93a75674-771f-42db-996f-b6f244100914/4411e000-ae8c-47f9-a8af-5ab99a6a34d5"
-					(reference "#PWR05")
+					(reference "#PWR?")
 					(unit 1)
 				)
@@
 		(dnp no)
 		(fields_autoplaced yes)
-		(property "Reference" "#PWR04"
+		(property "Reference" "#PWR?"
 			(at 104.14 102.87 0)
 			(hide yes)
@@
 			(project "Projeto_2_Microcontrolador_ponteH"
 				(path "/93a75674-771f-42db-996f-b6f244100914/4411e000-ae8c-47f9-a8af-5ab99a6a34d5"
-					(reference "#PWR04")
+					(reference "#PWR?")
 					(unit 1)
 				)
@@
 		(dnp no)
 		(fields_autoplaced yes)
-		(property "Reference" "C1"
+		(property "Reference" "C?"
 			(at 107.95 82.5499 0)
 			(show_name no)
@@
 			(project "Projeto_2_Microcontrolador_ponteH"
 				(path "/93a75674-771f-42db-996f-b6f244100914/4411e000-ae8c-47f9-a8af-5ab99a6a34d5"
-					(reference "C1")
+					(reference "C?")
 					(unit 1)
 				)
@@
 		(dnp no)
 		(fields_autoplaced yes)
-		(property "Reference" "C2"
+		(property "Reference" "C?"
 			(at 158.75 81.2799 0)
 			(show_name no)
@@
 			(project "Projeto_2_Microcontrolador_ponteH"
 				(path "/93a75674-771f-42db-996f-b6f244100914/4411e000-ae8c-47f9-a8af-5ab99a6a34d5"
-					(reference "C2")
-					(unit 1)
-				)
+					(reference "C?")
+					(unit 1)
+				)

Commit message: Atualização
Parts:
- added U2: TLV70433DBVR, Package_TO_SOT_SMD:SOT-23-5, symbol Project2_Symbols:TLV70433DBVR
Connections:
- net 12V_IN: now also U2.2 (IN)
- net 3V3_OUT: now also U2.3 (OUT)
- net GND: now also U2.1 (GND), U2.4 (NC), U2.5 (NC)
Other:
- note removed: "Create TLV704 Symbol"
