File: Projeto_2_Microcontrolador_ponteH/motor.kicad_sch (KiCad schematic)
At the start: 0 parts

Commit message: Atualização
Parts:
- added C? (x2): C, symbol Device:C
- added C?: C_Polarized, symbol Device:C_Polarized
- added J1: Screw_Terminal_01x02, symbol Connector:Screw_Terminal_01x02
Other:
- note added: "PT2466"

Commit message: Atualização
Parts:
- added C1: C, symbol Device:C
- added U1: PT2466, Package_SO:SOP-8_3.76x4.96mm_P1.27mm, symbol Project2_Symbols:PT2466
Connections:
- net MT_IN1: now also U1.6 (IN1)
- net MT_IN2: now also U1.5 (IN2)
- net MT_~{SLEEP}: now also U1.7 (nSLEEP)
- net +3V3: now reaches C?.1
- net +3V3: now also U1.8 (VCC)
- net GND: now reaches C?.2
- net GND: now also C?.2, C?.2, U1.4 (GND)
- net at J1.1 (Pin_1): now also C1.1, U1.2 (OUT1)
- net at J1.2 (Pin_2): now also C1.2, U1.3 (OUT2)
- net +12V: now reaches C?.1
- net +12V: now also C?.1, U1.1 (VM)
Other:
- note removed: "PT2466"
- moved on the sheet: C?, J1
